Commit message: Move robot back to 0,0,0

File: docker/robot_cell/robot_cell_support/urdf/robot_cell.xacro (robot description, xacro)
@@ -7,5 +7,5 @@
         <parent link="world" />
         <child link="base_link" />
-        <origin xyz="0.5 0 0" rpy="0 0 0"/>
+        <origin xyz="0 0 0" rpy="0 0 0"/>
     </joint>
 </robot>
